File: fluidics-v2/syrpump.kicad_sch (KiCad schematic)
At the start: 7 parts, among them U11 MAX3221

Commit message: V3: strip to minimal fluidics config, add 6th selector valve, fix lib paths
Reduce the V2 fluidics controller to a minimal build and extend the
selector-valve bank:

- Remove disc-pump driver (U1, M1); keep the syringe pump only
- Remove the solenoid-valve subsystem (MCZ33996 IC1 + D5-D20 + R6-R21
  + connector J5) -- 16 solenoids -> 0
- Remove all SPI pressure sensors (IC3-IC6 and their passives) -- 4 -> 0
- Reduce I2C flow sensors 4 -> 3 (drop connector J17)
- Add a 6th IDEX selector-valve channel (connectors J24/J25) on the
  shared isolated-I2C + 24V bus
- Remove the Wenzel-lab pressure-controller daughter board interface
  (J6, J7/ICSP, J8, JP3)
- Remove the manual-control block (switches S1-S4, push-button SW1,
  potentiometer VR1, TCA9539 U7, pull-ups, jumpers)
- Remove the 24V->12V converter (U5 + indicator D1/R2 + power-good R52);
  no remaining 12V load after the above

Net component count: 177 -> 86 footprints. DRC: 0 unconnected.

Tooling/portability fixes:
- Rewrite fp-lib-table and sym-lib-table: replace the original author's
  hardcoded absolute paths (/home/octopi-codex/...) with ${KIPRJMOD}-
  relative URIs so the libraries resolve on any machine
- Migrate the project to KiCad 10 format
- Add .gitignore for KiCad lock/autosave/cache and editor history files
- Add fluidics-v3-schematic.pdf (rendered schematic for review)

Co-Authored-By: Claude Opus 4.8 (1M context) <noreply@anthropic.com>
Parts:
- gave numbers to parts that had none: 6
