File: fluidics-v2/bubblesensors.kicad_sch (KiCad schematic)
At the start: 6 parts, among them U12 CD4050BDR, U13 TC7PZ17FU

Commit message: V3: strip to minimal fluidics config, add 6th selector valve, fix lib paths
Reduce the V2 fluidics controller to a minimal build and extend the
selector-valve bank:

- Remove disc-pump driver (U1, M1); keep the syringe pump only
- Remove the solenoid-valve subsystem (MCZ33996 IC1 + D5-D20 + R6-R21
  + connector J5) -- 16 solenoids -> 0
- Remove all SPI pressure sensors (IC3-IC6 and their passives) -- 4 -> 0
- Reduce I2C flow sensors 4 -> 3 (drop connector J17)
- Add a 6th IDEX selector-valve channel (connectors J24/J25) on the
  shared isolated-I2C + 24V bus
- Remove the Wenzel-lab pressure-controller daughter board interface
  (J6, J7/ICSP, J8, JP3)
- Remove the manual-control block (switches S1-S4, push-button SW1,
  potentiometer VR1, TCA9539 U7, pull-ups, jumpers)
- Remove the 24V->12V converter (U5 + indicator D1/R2 + power-good R52);
  no remaining 12V load after the above

Net component count: 177 -> 86 footprints. DRC: 0 unconnected.

Tooling/portability fixes:
- Rewrite fp-lib-table and sym-lib-table: replace the original author's
  hardcoded absolute paths (/home/octopi-codex/...) with ${KIPRJMOD}-
  relative URIs so the libraries resolve on any machine
- Migrate the project to KiCad 10 format
- Add .gitignore for KiCad lock/autosave/cache and editor history files
- Add fluidics-v3-schematic.pdf (rendered schematic for review)

Co-Authored-By: Claude Opus 4.8 (1M context) <noreply@anthropic.com>
Parts:
- gave numbers to parts that had none: 4

Commit message: @ Wire solenoid driver + status LEDs + I2C cleanup; route + connect
- Solenoid driver (U1 TPL7407): IN1-7 <- Teensy GPIO_1-7 (back-layer fanout,
  vias off the SMD pads), COM->+24V, GND->plane, OUT1-7 -> J5 screw terminal
- Add 7 solenoid status LEDs (GPIO_1-7) + COM/+24V indicator LED (0402)
- Remove LTC4311 I2C accelerators (U9/U10) - misbehaved on lightly-loaded
  buses (single-valve failure); kept passive pull-ups. Restored SCL2/SDA2
  pull-ups (R41/R42)
- Back layer: full-board GND pour (clean rectangle outline)
- Connect U1 GND and R4 (+24V power-indicator LED) to their nets

DRC: unconnected down to 5, all intentional unused-pin no-connects
(GPIO_8/9 + vestigial SPI). No shorts; vias cleared out of Teensy SMD pads.

Co-Authored-By: Claude Opus 4.8 (1M context) <noreply@anthropic.com>
@
Parts:
- U12: footprint D16 -> hexbuf:D16
- U13: footprint SOT-363 US6_TOS -> TC7PZ17FU:SOT-363 US6_TOS
Changed lines of the file:
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@@
 			)
 		)
-		(property "Footprint" "SOT-363   US6_TOS"
+		(property "Footprint" "TC7PZ17FU:SOT-363   US6_TOS"
 			(at 41.91 22.86 0)
 			(hide yes)
@@
 			)
 		)
-		(property "Footprint" "D16"
+		(property "Footprint" "hexbuf:D16"
 			(at 40.64 76.2 0)
 			(hide yes)
