File: fluidics-v2/manualctrl.kicad_sch (KiCad schematic)
At the start: 26 parts, among them SW1 D6C90F1LFS, U7 TCA9539PWR

Commit message: V3: strip to minimal fluidics config, add 6th selector valve, fix lib paths
Reduce the V2 fluidics controller to a minimal build and extend the
selector-valve bank:

- Remove disc-pump driver (U1, M1); keep the syringe pump only
- Remove the solenoid-valve subsystem (MCZ33996 IC1 + D5-D20 + R6-R21
  + connector J5) -- 16 solenoids -> 0
- Remove all SPI pressure sensors (IC3-IC6 and their passives) -- 4 -> 0
- Reduce I2C flow sensors 4 -> 3 (drop connector J17)
- Add a 6th IDEX selector-valve channel (connectors J24/J25) on the
  shared isolated-I2C + 24V bus
- Remove the Wenzel-lab pressure-controller daughter board interface
  (J6, J7/ICSP, J8, JP3)
- Remove the manual-control block (switches S1-S4, push-button SW1,
  potentiometer VR1, TCA9539 U7, pull-ups, jumpers)
- Remove the 24V->12V converter (U5 + indicator D1/R2 + power-good R52);
  no remaining 12V load after the above

Net component count: 177 -> 86 footprints. DRC: 0 unconnected.

Tooling/portability fixes:
- Rewrite fp-lib-table and sym-lib-table: replace the original author's
  hardcoded absolute paths (/home/octopi-codex/...) with ${KIPRJMOD}-
  relative URIs so the libraries resolve on any machine
- Migrate the project to KiCad 10 format
- Add .gitignore for KiCad lock/autosave/cache and editor history files
- Add fluidics-v3-schematic.pdf (rendered schematic for review)

Co-Authored-By: Claude Opus 4.8 (1M context) <noreply@anthropic.com>
Parts:
- removed C?: 0.1u, Capacitor_SMD:C_0603_1608Metric, symbol Device:C
- removed C?: 1u, Capacitor_SMD:C_0805_2012Metric, symbol Device:C
- removed JP1, JP2: SolderJumper_3_Bridged12, Jumper:SolderJumper-3_P1.3mm_Bridged12_Pad1.0x1.5mm_NumberLabels, symbol Jumper:SolderJumper_3_Bridged12
- removed R24, R25, R26, R27, R28, R29, R30, R31, R32, R33, R34, R35, R36, R37, R38: 10k, Resistor_SMD:R_0402_1005Metric, symbol Device:R
- removed S1, S4: 210-6MS, 210-6MS:2106MS, symbol 210-6MS:210-6MS
- removed S2, S3: 450301014042, wurth:450301014042, symbol 450301014042:450301014042
- removed SW1: D6C90F1LFS, SW4_D6C90F1LFS_CNK, symbol SW4_D6C90F1LFS_CNK:D6C90F1LFS
- removed U7: TCA9539PWR, TCA9539PWR:PW24, symbol 2023-08-08_01-32-38:TCA9539PWR
- removed VR1: PTV09A-4020U-B103, bourns:PTV09A4015FB103, symbol bourns:PTV09A-4020U-B103
Connections:
- no-connect marks 3 -> 0
Other:
- note removed: ""Set Valves" momentary pushbutton"
- note removed: "12 DIP switches Control up to 12 valves independently"
- note removed: "14 input devices - 12 DIP switches, 1 switch, 1 button"
- note removed: "Enable/Disable Manual Control"
- note removed: "GPIO expander Connect to 12 DIP switches, 1 switch, 1 button over I2C (all inputs)"
- note removed: "Potentiometer for manual pump control"
- note removed: "Pressure/Vacuum selector (sets valves 1/4 to either be both on or both off)"
- note removed: "Use solder jumpers to set the address Default = 0x74"

Commit message: @ Wire solenoid driver + status LEDs + I2C cleanup; route + connect
- Solenoid driver (U1 TPL7407): IN1-7 <- Teensy GPIO_1-7 (back-layer fanout,
  vias off the SMD pads), COM->+24V, GND->plane, OUT1-7 -> J5 screw terminal
- Add 7 solenoid status LEDs (GPIO_1-7) + COM/+24V indicator LED (0402)
- Remove LTC4311 I2C accelerators (U9/U10) - misbehaved on lightly-loaded
  buses (single-valve failure); kept passive pull-ups. Restored SCL2/SDA2
  pull-ups (R41/R42)
- Back layer: full-board GND pour (clean rectangle outline)
- Connect U1 GND and R4 (+24V power-indicator LED) to their nets

DRC: unconnected down to 5, all intentional unused-pin no-connects
(GPIO_8/9 + vestigial SPI). No shorts; vias cleared out of Teensy SMD pads.

Co-Authored-By: Claude Opus 4.8 (1M context) <noreply@anthropic.com>
@
Other:
- note added: "Add extra components here, if needed."
Changed lines of the file:
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@@
 	(generator_version "10.0")
 	(paper "A4")
+	(text "Add extra components here, if needed. "
+		(exclude_from_sim no)
+		(at 200.152 173.99 0)
+		(effects
+			(font
+				(size 1.27 1.27)
+				(thickness 0.1588)
+			)
+		)
+	)
 )
