File: fluidics-v2/psu.kicad_sch (KiCad schematic)
At the start: 15 parts, among them U3 AP7366EA-33W5-7, U4 D24V10FX

Commit message: V3: strip to minimal fluidics config, add 6th selector valve, fix lib paths
Reduce the V2 fluidics controller to a minimal build and extend the
selector-valve bank:

- Remove disc-pump driver (U1, M1); keep the syringe pump only
- Remove the solenoid-valve subsystem (MCZ33996 IC1 + D5-D20 + R6-R21
  + connector J5) -- 16 solenoids -> 0
- Remove all SPI pressure sensors (IC3-IC6 and their passives) -- 4 -> 0
- Reduce I2C flow sensors 4 -> 3 (drop connector J17)
- Add a 6th IDEX selector-valve channel (connectors J24/J25) on the
  shared isolated-I2C + 24V bus
- Remove the Wenzel-lab pressure-controller daughter board interface
  (J6, J7/ICSP, J8, JP3)
- Remove the manual-control block (switches S1-S4, push-button SW1,
  potentiometer VR1, TCA9539 U7, pull-ups, jumpers)
- Remove the 24V->12V converter (U5 + indicator D1/R2 + power-good R52);
  no remaining 12V load after the above

Net component count: 177 -> 86 footprints. DRC: 0 unconnected.

Tooling/portability fixes:
- Rewrite fp-lib-table and sym-lib-table: replace the original author's
  hardcoded absolute paths (/home/octopi-codex/...) with ${KIPRJMOD}-
  relative URIs so the libraries resolve on any machine
- Migrate the project to KiCad 10 format
- Add .gitignore for KiCad lock/autosave/cache and editor history files
- Add fluidics-v3-schematic.pdf (rendered schematic for review)

Co-Authored-By: Claude Opus 4.8 (1M context) <noreply@anthropic.com>
Parts:
- removed D1: LED, LED_SMD:LED_0805_2012Metric_Pad1.15x1.40mm_HandSolder, symbol Device:LED
- removed R2: 20k, Resistor_SMD:R_0603_1608Metric_Pad0.98x0.95mm_HandSolder, symbol Device:R
- removed R52: 47k, Resistor_SMD:R_0603_1608Metric_Pad0.98x0.95mm_HandSolder, symbol Device:R
- removed U5: ~, D36V28Fx:D36V28Fx, symbol D36V28Fx:D36V28FX
Connections:
- no-connect marks 2 -> 1
Other:
- note removed: "24V -> 12V for selector valves"

Commit message: @ Wire solenoid driver + status LEDs + I2C cleanup; route + connect
- Solenoid driver (U1 TPL7407): IN1-7 <- Teensy GPIO_1-7 (back-layer fanout,
  vias off the SMD pads), COM->+24V, GND->plane, OUT1-7 -> J5 screw terminal
- Add 7 solenoid status LEDs (GPIO_1-7) + COM/+24V indicator LED (0402)
- Remove LTC4311 I2C accelerators (U9/U10) - misbehaved on lightly-loaded
  buses (single-valve failure); kept passive pull-ups. Restored SCL2/SDA2
  pull-ups (R41/R42)
- Back layer: full-board GND pour (clean rectangle outline)
- Connect U1 GND and R4 (+24V power-indicator LED) to their nets

DRC: unconnected down to 5, all intentional unused-pin no-connects
(GPIO_8/9 + vestigial SPI). No shorts; vias cleared out of Teensy SMD pads.

Co-Authored-By: Claude Opus 4.8 (1M context) <noreply@anthropic.com>
@
Parts:
- D2, D3, D4: footprint LED_SMD:LED_0805_2012Metric_Pad1.15x1.40mm_HandSolder -> LED_SMD:LED_0805_2012Metric
- R3: footprint Resistor_SMD:R_0603_1608Metric_Pad0.98x0.95mm_HandSolder -> Resistor_SMD:R_0805_2012Metric
- R4, R5: footprint Resistor_SMD:R_0603_1608Metric_Pad0.98x0.95mm_HandSolder -> Resistor_SMD:R_0402_1005Metric
Changed lines of the file:
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@@
 			)
 		)
-		(property "Footprint" "LED_SMD:LED_0805_2012Metric_Pad1.15x1.40mm_HandSolder"
+		(property "Footprint" "LED_SMD:LED_0805_2012Metric"
 			(at 90.17 59.69 0)
 			(hide yes)
@@
 			)
 		)
-		(property "Footprint" "LED_SMD:LED_0805_2012Metric_Pad1.15x1.40mm_HandSolder"
+		(property "Footprint" "LED_SMD:LED_0805_2012Metric"
 			(at 101.6 59.69 0)
 			(hide yes)
@@
 			)
 		)
-		(property "Footprint" "Resistor_SMD:R_0603_1608Metric_Pad0.98x0.95mm_HandSolder"
+		(property "Footprint" "Resistor_SMD:R_0805_2012Metric"
 			(at 88.392 52.07 90)
 			(hide yes)
@@
 			)
 		)
-		(property "Footprint" "Resistor_SMD:R_0603_1608Metric_Pad0.98x0.95mm_HandSolder"
+		(property "Footprint" "Resistor_SMD:R_0402_1005Metric"
 			(at 99.822 52.07 90)
 			(hide yes)
@@
 			)
 		)
-		(property "Footprint" "LED_SMD:LED_0805_2012Metric_Pad1.15x1.40mm_HandSolder"
+		(property "Footprint" "LED_SMD:LED_0805_2012Metric"
 			(at 111.76 59.69 0)
 			(hide yes)
@@
 			)
 		)
-		(property "Footprint" "Resistor_SMD:R_0603_1608Metric_Pad0.98x0.95mm_HandSolder"
+		(property "Footprint" "Resistor_SMD:R_0402_1005Metric"
 			(at 109.982 52.07 90)
 			(hide yes)
