File: fluidics-v2/sensors.kicad_sch (KiCad schematic)
At the start: 27 parts, among them IC3 HSCDRRN001BDSA3, IC4 HSCDRRN001BDSA3, IC5 HSCDRRN001BDSA3, IC6 HSCDRRN001BDSA3, U16 LTC4316CMS-TRPBF

Commit message: V3: strip to minimal fluidics config, add 6th selector valve, fix lib paths
Reduce the V2 fluidics controller to a minimal build and extend the
selector-valve bank:

- Remove disc-pump driver (U1, M1); keep the syringe pump only
- Remove the solenoid-valve subsystem (MCZ33996 IC1 + D5-D20 + R6-R21
  + connector J5) -- 16 solenoids -> 0
- Remove all SPI pressure sensors (IC3-IC6 and their passives) -- 4 -> 0
- Reduce I2C flow sensors 4 -> 3 (drop connector J17)
- Add a 6th IDEX selector-valve channel (connectors J24/J25) on the
  shared isolated-I2C + 24V bus
- Remove the Wenzel-lab pressure-controller daughter board interface
  (J6, J7/ICSP, J8, JP3)
- Remove the manual-control block (switches S1-S4, push-button SW1,
  potentiometer VR1, TCA9539 U7, pull-ups, jumpers)
- Remove the 24V->12V converter (U5 + indicator D1/R2 + power-good R52);
  no remaining 12V load after the above

Net component count: 177 -> 86 footprints. DRC: 0 unconnected.

Tooling/portability fixes:
- Rewrite fp-lib-table and sym-lib-table: replace the original author's
  hardcoded absolute paths (/home/octopi-codex/...) with ${KIPRJMOD}-
  relative URIs so the libraries resolve on any machine
- Migrate the project to KiCad 10 format
- Add .gitignore for KiCad lock/autosave/cache and editor history files
- Add fluidics-v3-schematic.pdf (rendered schematic for review)

Co-Authored-By: Claude Opus 4.8 (1M context) <noreply@anthropic.com>
Parts:
- removed C? (x4): 0.1u, Capacitor_SMD:C_0603_1608Metric, symbol Device:C
- removed C? (x4): 1u, Capacitor_SMD:C_0805_2012Metric, symbol Device:C
- removed IC3, IC4, IC5, IC6: HSCDRRN001BDSA3, HSCDRRN001BDSA3:HSCDRRN001BDSA3, symbol HSCDRRN001BDSA3:HSCDRRN001BDSA3
- removed R56, R57, R58, R59: 4.7k, Resistor_SMD:R_0402_1005Metric, symbol Device:R
- gave numbers to parts that had none: 2
Connections:
- no-connect marks 13 -> 1

Commit message: @ WIP: continue strip-down — empty sensors sheet, drop 11 PCB footprints
Recovered in-progress work from the previous KiCad session (restored via
KiCad session recovery). This is mid-edit, not a finished config:
- sensors.kicad_sch: 17 -> 0 symbols (sheet fully emptied)
- fluidics-v2.kicad_pcb: 86 -> 75 footprints
- fluidics-v2.kicad_sch: minor net/sheet cleanup

Schematic + libraries validated with kicad-cli sch export netlist (exit 0).

Co-Authored-By: Claude Opus 4.8 (1M context) <noreply@anthropic.com>
@
Parts:
- removed C30: 0.1u, Capacitor_SMD:C_0603_1608Metric, symbol Device:C
- removed C35: 1u, Capacitor_SMD:C_0805_2012Metric, symbol Device:C
- removed JP4, JP5: SolderJumper_2_Open, Jumper:SolderJumper-2_P1.3mm_Open_TrianglePad1.0x1.5mm, symbol Jumper:SolderJumper_2_Open
- removed R45: 976k, Resistor_SMD:R_0603_1608Metric_Pad0.98x0.95mm_HandSolder, symbol Device:R
- removed R46: DNP, Resistor_SMD:R_0603_1608Metric_Pad0.98x0.95mm_HandSolder, symbol Device:R
- removed R47: 102k, Resistor_SMD:R_0603_1608Metric_Pad0.98x0.95mm_HandSolder, symbol Device:R
- removed R48: 0, Resistor_SMD:R_0603_1608Metric_Pad0.98x0.95mm_HandSolder, symbol Device:R
- removed R49, R50: 4.7k, Resistor_SMD:R_0402_1005Metric, symbol Device:R
- removed U16: LTC4316CMS-TRPBF, addresstranslator:MSOP-10_MS_LIT, symbol LTC4316CMS:LTC4316CMS-TRPBF
Connections:
- no-connect marks 1 -> 0
Other:
- note removed: "Address translator for fourth flow sensor - DNP if using only three If the translator is not populated, connect the solder jumpers to use 4th connector"
- note removed: "Change resistor values to set the new address See page 9: https://www.analog.com/media/en/technical-documentation/data-sheets/4316fa.pdf"
- note removed: "Only one device on bus - use a larger resistor"
- note removed: "Pressure sensors connect over SPI and have unique chip select pins"

Commit message: @ Wire solenoid driver + status LEDs + I2C cleanup; route + connect
- Solenoid driver (U1 TPL7407): IN1-7 <- Teensy GPIO_1-7 (back-layer fanout,
  vias off the SMD pads), COM->+24V, GND->plane, OUT1-7 -> J5 screw terminal
- Add 7 solenoid status LEDs (GPIO_1-7) + COM/+24V indicator LED (0402)
- Remove LTC4311 I2C accelerators (U9/U10) - misbehaved on lightly-loaded
  buses (single-valve failure); kept passive pull-ups. Restored SCL2/SDA2
  pull-ups (R41/R42)
- Back layer: full-board GND pour (clean rectangle outline)
- Connect U1 GND and R4 (+24V power-indicator LED) to their nets

DRC: unconnected down to 5, all intentional unused-pin no-connects
(GPIO_8/9 + vestigial SPI). No shorts; vias cleared out of Teensy SMD pads.

Co-Authored-By: Claude Opus 4.8 (1M context) <noreply@anthropic.com>
@
Other:
- note added: "Subsheet for extra sensors. Add those sensors here, if needed."
Changed lines of the file:
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@@
 	(generator_version "10.0")
 	(paper "A4")
+	(text "Subsheet for extra sensors. Add those sensors here, if needed. "
+		(exclude_from_sim no)
+		(at 210.566 173.736 0)
+		(effects
+			(font
+				(size 1.27 1.27)
+				(thickness 0.1588)
+			)
+		)
+	)
 )
