File: fluidics-v2/fluidics-v2.kicad_pcb (KiCad board)
At the start: 4 copper layers, 82.5 x 95.5 mm, 76 parts, among them IC2 ADUM1250WSRZ-RL7, J1 PJ-063AH, J10 87832-1010, J11 0705430001, J12 87832-1010, J13 0705430001, J14 87832-1010, J15 0533980671, J16 0705430001, J17 0533980671, J18 87832-1010, J19 0705430001, J2 B6B-ZR-SM4-TF, J20 0533980671, J21 87832-1010, J22 0705430001, J24 0705430001, J25 87832-1010, J3 A-DS_15_A_KG-T4S, J4 B6B-ZR-SM4-TF, J5 Screw_Terminal_01x02, J6 Screw_Terminal_01x02, U1 TPL7407LDR, U11 MAX3221, U12 CD4050BDR, U13 TC7PZ17FU, U2 Teensy4.1, U3 AP7366EA-33W5-7, U4 D24V10FX, U6 LTC4311CSC6-TRPBF

Commit message: PCB fix: add R1 (svalves), clear dangling track; refresh schematic PDF
- Add resistor R1 on svalves sheet, placed on board; footprints 76 -> 77.
- Prior dangling J6 track resolved (DRC track_dangling now 0).
- DRC: schematic_parity 0, 5 intentional no-connects, rest cosmetic
  (silk/courtyard/padstack inherited from upstream).
- Regenerate fluidics-v3-schematic.pdf from current schematic.

Co-Authored-By: Claude Opus 4.8 (1M context) <noreply@anthropic.com>
Parts:
- added R1: 0, Resistor_SMD:R_0402_1005Metric, F.Cu at (129.5, 36.0)
- moved TP3 2.81 mm to (132.5, 37.0)
Routing:
- net /Selector Valves/SCL 5V: track 117.4 -> 122.1 mm, vias 1 -> 3
- net /Selector Valves/SDA 5V: track 105.4 -> 109.7 mm
- net GND: track 134.6 -> 133.2 mm
