File: fluidics-v3/fluidics-v3.kicad_sch (KiCad schematic)
At the start: 41 parts, among them J1 PJ-063AH, J10 87832-0410, J11 0705430001, J12 87832-0410, J13 0705430001, J14 87832-0410, J15 0533980671, J16 0705430001, J17 0533980671, J18 87832-0410, J19 0705430001, J2 B6B-ZR-SM4-TF, J20 0533980671, J21 87832-0410, J22 0705430001, J24 0705430001, J25 87832-0410, J3 A-DS_15_A_KG-T4S, J4 B6B-ZR-SM4-TF, J6 SSM-124-L-SV, J7 SSM-124-L-SV, U2 Teensy4.1

Commit message: v3: +24V soft-start front end, U1 COM bypass, silkscreen and BOM fixes
Power input stage
- Replace TH1 (10 ohm NTC) with a low-side N-channel soft-start: Q1 (F60N80,
  TO-220) with a 100k/68k gate divider (R2/R6) and 0.1u timing cap (C11).
  The NTC sat in series with the whole board and dissipated 1.5-10 W; at
  1.85 A it was already over a 7 mm disc's rating before any valve moved.
- Split ground: /GND1 (J1 shell + pin 2) is now separate from GND, with Q1
  bridging them. Removed a leftover 2.39 mm GND track that still touched
  J1.S2 and shorted straight across Q1.
- Add C12 470u/50V bulk and C13 0.1u HF bypass on +24V. C3 alone left the
  300 kHz - 100 MHz band uncovered while U4 switches at 500 kHz.
- Route the block: gate net kept inside 5 mm of Q1's gate; /GND1 return at
  1.50 mm (4.3 A capacity vs 1.85 A worst case through Q1).

Solenoid driver
- Add C25 0.1u across U1 pin 9 (COM) to GND. That node catches flyback from
  all seven channels and previously reached the +24V plane through ~50 mm of
  0.55 mm trace with nothing local.

Silkscreen
- Raise 403 graphic objects from 0.000/0.100/0.120/0.127 mm to the 0.15 mm
  fab minimum; five were zero-width, which is undefined behaviour. Fix one
  0.45 mm text height and one 0.09 mm stroke.
- Selector valve legend: label 'J23' named a part that does not exist; the
  connector there is J25. Recentre all 12 labels on their own connectors,
  strip stray newlines, and hide 7 duplicate footprint refdes that sat
  midway between connectors and read as shifted by one.

Cleanup
- Remove two /SDA and /SCL vias that connected B.Cu to B.Cu after those nets
  moved to the back layer, and split a +3.3V track so its end meets a
  junction rather than landing mid-span.
- Stitch an orphaned F.Cu ground island that had captured D3's cathode pad.

BOM
- Correct three MPNs that contradicted their own values and packages:
  R3 5.6k/0805 was a 680R 0603 part, R4 47k/0402 was a 4k7 0603 part,
  R5 3k/0402 was a 270R 0603 part.
- J1 car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
Parts:
- removed TH1: 10R, Varistor:RV_Disc_D7mm_W3.9mm_P5mm, symbol Device:Thermistor_NTC
- added C11, C13: 0.1u, Capacitor_SMD:C_0603_1608Metric, symbol Device:C
- added C12: 470u 50V, Capacitor_THT:CP_Radial_D10.0mm_P5.00mm, symbol Device:C_Polarized
- added Q1: F60N80, Package_TO_SOT_THT:TO-220-3_Vertical, symbol Transistor_FET:Q_NMOS_GDS
- added R2: 100k, Resistor_SMD:R_0402_1005Metric, symbol Device:R
- added R6: 68k, Resistor_SMD:R_0402_1005Metric, symbol Device:R
- J1: MANUFACTURER CUI INC -> (none); Manufacturer_Name (none) -> CUI Devices; Manufacturer_Part_Number (none) -> PJ-063AH
- J15, J17, J20: MANUFACTURER Molex -> (none); Manufacturer_Name (none) -> Molex
- J2, J4: MANUFACTURER JST -> (none); Manufacturer_Name (none) -> JST
- R10: value 47K -> 47k
- R11, R12, R9: value 2.7K -> 2.7k
Connections:
- net +24V_IN is gone; now on net +24V: J1.1
- net +24V: now also C12.1, C13.1, R2.1
- net GND: now also C12.2, C13.2, Q1.2 (D); no longer J1.2, J1.S1 (SHIELD), J1.S2 (SHIELD__1)
- net PG-12V: no longer U2.24 (32_OUT1B)
- net SCL: now also J20.2, J7.17 (Pin_17), TP1.1, U2.41 (19_A5_SCL); no longer J20.5, J7.16 (Pin_16), TP1.2, U2.40 (18_A4_SDA)
- net SDA: now also J20.5, J7.16 (Pin_16), TP1.2, U2.40 (18_A4_SDA); no longer J20.2, J7.17 (Pin_17), TP1.1, U2.41 (19_A5_SCL)
- new net: C11.1, Q1.1 (G), R2.2, R6.1
- new net GND1: C11.2, J1.2, J1.S1 (SHIELD), J1.S2 (SHIELD__1), Q1.3 (S), R6.2
- no-connect marks 53 -> 54
Other:
- removed sheet Sensors
- sheet Power Supplies ports: added none; removed PG-12V
- sheet Solenoid Valve Driver ports: added none; removed GPIO_1, GPIO_2, GPIO_3, GPIO_4
- note added: "Bulk Electrolytic Bypasses"
- note added: "NMOS Soft Start Network with Bypass Capacitors"
- note removed: "Convert from 24V to: - 12V - 5V - 3.3V"
- moved on the sheet: C10, C3, C4, D10, D11, D12, D9, H2, H3, H4, J1, J10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

Commit message: fab: reconcile BOM against CPL for assembly
The assembler rejected 17 designators as "not in the BOM" and 24 as "not in
the CPL". Two separate causes:

Reference ranges
- The BOM collapsed runs into ranges (C15-C17, D9-D12, H2-H4, R39-R44).
  Assembly parsers read those literally, so every designator inside a range
  looked absent. Export with --ref-range-delimiter '' so each one is listed.

Parts that are in the BOM but cannot be placed
- H2-H4 (mounting holes) and TP1-TP3 (test points) carry the
  "exclude from position files" footprint attribute, so they never reach the
  CPL, but were still marked in_bom. They are not parts; set in_bom no.
- U2 (Teensy 4.1) has on_board no - it plugs into sockets J6/J7 and has no
  footprint, so it cannot appear in a CPL either. Excluded from the assembly
  BOM; the module itself is still documented in README as a separate item.

BOM and CPL now list the same 78 designators, with no ranges and no
one-sided entries. ERC: 0 errors.

Co-Authored-By: Claude Opus 5 (1M context) <noreply@anthropic.com>
Parts:
- H2, H3, H4, TP1, TP2, TP3, U2: now left out of the parts list
Changed lines of the file:
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@@
 		(body_style 1)
 		(exclude_from_sim no)
-		(in_bom yes)
+		(in_bom no)
 		(on_board yes)
 		(in_pos_files no)
@@
 		(body_style 1)
 		(exclude_from_sim no)
-		(in_bom yes)
+		(in_bom no)
 		(on_board yes)
 		(in_pos_files no)
@@
 		(body_style 1)
 		(exclude_from_sim no)
-		(in_bom yes)
+		(in_bom no)
 		(on_board yes)
 		(in_pos_files no)
@@
 		(body_style 1)
 		(exclude_from_sim no)
-		(in_bom yes)
+		(in_bom no)
 		(on_board no)
 		(in_pos_files yes)
@@
 		(body_style 1)
 		(exclude_from_sim no)
-		(in_bom yes)
+		(in_bom no)
 		(on_board yes)
 		(in_pos_files no)
@@
 		(body_style 1)
 		(exclude_from_sim no)
-		(in_bom yes)
+		(in_bom no)
 		(on_board yes)
 		(in_pos_files no)
@@
 		(body_style 1)
 		(exclude_from_sim no)
-		(in_bom yes)
+		(in_bom no)
 		(on_board yes)
 		(in_pos_files no)

Commit message: fab: mark J6/J7 DNP - Teensy sockets are hand-fitted
J6 and J7 (SSM-124-L-SV) are sourced and soldered in-house, so the board
house should not fit them. Set dnp on both the symbols and the footprints
rather than "exclude from BOM", because DNP states the intent - the parts
belong on the board, the assembler just skips them - and both exporters
honour --exclude-dnp, which keeps the two files in step automatically.

Regenerated with --exclude-dnp on both sides:
- BOM  34 rows, 76 designators
- CPL  76 designators
- reconciled: nothing on one side only, no reference ranges

All 12 through-hole parts stay in (C12, J1, J3, J5, J11, J13, J16, J19,
J22, J24, Q1, U4) since THT assembly is being ordered.

The STEP model still contains J6/J7 - the sockets are physically present on
the finished board, and the board geometry itself did not change.

ERC: 0 errors. DRC: 0 errors, 0 unconnected, 0 parity.

Co-Authored-By: Claude Opus 5 (1M context) <noreply@anthropic.com>
Parts:
- J6, J7: now not fitted
Changed lines of the file:
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@@
 		(on_board yes)
 		(in_pos_files yes)
-		(dnp no)
+		(dnp yes)
 		(property "Reference" "J6"
 			(at 86.868 100.33 0)
@@
 		(on_board yes)
 		(in_pos_files yes)
-		(dnp no)
+		(dnp yes)
 		(fields_autoplaced yes)
 		(property "Reference" "J7"
