File: fluidics-v3/fluidics-v3.kicad_sch (KiCad schematic)
At the start: 46 parts, among them J1 PJ-063AH, J10 87832-0410, J11 0705430001, J12 87832-0410, J13 0705430001, J14 87832-0410, J15 0533980671, J16 0705430001, J17 0533980671, J18 87832-0410, J19 0705430001, J2 B6B-ZR-SM4-TF, J20 0533980671, J21 87832-0410, J22 0705430001, J24 0705430001, J25 87832-0410, J3 A-DS_15_A_KG-T4S, J4 B6B-ZR-SM4-TF, J6 SSM-124-L-SV, J7 SSM-124-L-SV, Q1 F60N80, U2 Teensy4.1

Commit message: fab: apply JLCPCB part selections to BOM, annotate strays, normalise CPL
Sourcing
- Write Manufacturer_Part_Number / Manufacturer_Name / LCSC for every part
  from the JLCPCB BOM-matching sheet. 33 of 34 BOM rows now carry an LCSC
  code; the exception is J10/J12/J14/J18/J21/J25 (Molex 87832-0410), which
  JLCPCB returned "No matches" for and still needs a part chosen.

Substitutions accepted from the sheet
- IC2  ADuM1250WSRZ-RL7 -> ISO1640BDR (TI). Verified pin-for-pin against the
  board: 1 VCC1, 2 SDA1, 3 SCL1, 4 GND1, 5 GND2, 6 SCL2, 7 SDA2, 8 VCC2.
- C3   -> KEMET T521X336M050ATE050, which is 33uF/50V, not 100uF. Value
  updated to match. The 50 V rating fixes the derating problem the old
  unrated 100uF tantalum had on a 24 V rail; 33uF is ample now that C12
  carries 470uF ten millimetres away. Note the part is case X (7343-43,
  4.3 mm tall) against a footprint named 7343-20 - the land pattern is
  identical, only the height differs, and nothing sits above it.
- Q1   -> IRF540NPBF, J3 -> Connfly DS1037, D4 -> KT-0805R, J5 -> XY308.
- U13's MPN arrived truncated from JLCPCB as "TC7PZ17FU,LJ(CT"; restored the
  closing parenthesis.

Annotation
- D2/D3/D4, R3/R4/R5 (psu sheet) and H2/H3/H4 (root) were still unannotated
  "D?"/"R?"/"H?" symbols, so the BOM exporter was auto-numbering them on each
  run and no field edit could reach them. Annotated from the PCB footprint
  UUID paths rather than by position - H3 and H4 turned out to be the reverse
  of what their schematic coordinates suggested.

CPL
- Rotations now emitted 0-360; KiCad wrote 27 of them as negative (-90).
- Coordinates to 4 dp, rotation to 2 dp.
- BOM and CPL reconcile at 76 designators, no ranges, nothing one-sided.

ERC: 0 errors.

Co-Authored-By: Claude Opus 5 (1M context) <noreply@anthropic.com>
Parts:
- C10: LCSC (none) -> C394395; Manufacturer_Name (none) -> Taiyo Yuden; Manufacturer_Part_Number (none) -> EMK325ABJ107MM-T
- C11, C13: LCSC (none) -> C14663; Manufacturer_Name (none) -> YAGEO; Manufacturer_Part_Number (none) -> CC0603KRX7R9BB104
- C12: LCSC (none) -> C2912407; Manufacturer_Name (none) -> Changzhou Huawei Elec; Manufacturer_Part_Number (none) -> KM1H471MG200A00CV016
- C3: value 100u -> 33u 50V; LCSC (none) -> C2158776; Manufacturer_Name (none) -> KEMET; Manufacturer_Part_Number (none) -> T521X336M050ATE050
- C4: LCSC (none) -> C96123; Manufacturer_Name (none) -> Samsung Electro-Mechanics; Manufacturer_Part_Number (none) -> CL31A476MPHNNNE
- D10, D11, D12, D9: LCSC (none) -> C160479; Manufacturer_Name (none) -> Lite-On; Manufacturer_Part_Number (none) -> LTST-C281KGKT
- D21: LCSC (none) -> C110486; Manufacturer_Name (none) -> Diodes Incorporated; Manufacturer_Part_Number (none) -> B340-13-F
- J1: LCSC C2928097 -> C22434582; Manufacturer_Name CUI Devices -> CUI
- J11, J13: LCSC C5349069 -> C127361; Manufacturer_Name Molex -> MOLEX; Manufacturer_Part_Number 0705430001 -> 705430001
- J15, J17, J20: LCSC (none) -> C277393; Manufacturer_Name Molex -> MOLEX; Manufacturer_Part_Number (none) -> 533980671
- J16, J19, J22, J24: LCSC (none) -> C127361; Manufacturer_Name Molex -> MOLEX; Manufacturer_Part_Number 0705430001 -> 705430001
- J2, J4: LCSC (none) -> C471473; Manufacturer_Part_Number (none) -> B6B-ZR-SM4-TF(LF)(SN)
- J3: LCSC C3100941 -> C77837; Manufacturer_Name ASSMANN WSW components GmbH -> CONNFLY Elec; Manufacturer_Part_Number A-DS 15 A/KG-T4S -> DS1037-15MNCKT74-0CC
- Q1: LCSC (none) -> C2566; Manufacturer_Name (none) -> Infineon Technologies; Manufacturer_Part_Number (none) -> IRF540NPBF
- R10: LCSC (none) -> C25819; Manufacturer_Name (none) -> UNI-ROYAL(Uniroyal Elec); Manufacturer_Part_Number (none) -> 0603WAF4702T5E
- R11, R12, R9: LCSC (none) -> C25885; Manufacturer_Name (none) -> UNI-ROYAL(Uniroyal Elec); Manufacturer_Part_Number (none) -> 0402WGF2701TCE
- R2: LCSC (none) -> C25741; Manufacturer_Name (none) -> UNI-ROYAL(Uniroyal Elec); Manufacturer_Part_Number (none) -> 0402WGF1003TCE
- R6: LCSC (none) -> C36871; Manufacturer_Name (none) -> UNI-ROYAL(Uniroyal Elec); Manufacturer_Part_Number (none) -> 0402WGF6802TCE
