File: fluidics-v3/i2c.kicad_sch (KiCad schematic)
At the start: 2 parts

Commit message: v3: +24V soft-start front end, U1 COM bypass, silkscreen and BOM fixes
Power input stage
- Replace TH1 (10 ohm NTC) with a low-side N-channel soft-start: Q1 (F60N80,
  TO-220) with a 100k/68k gate divider (R2/R6) and 0.1u timing cap (C11).
  The NTC sat in series with the whole board and dissipated 1.5-10 W; at
  1.85 A it was already over a 7 mm disc's rating before any valve moved.
- Split ground: /GND1 (J1 shell + pin 2) is now separate from GND, with Q1
  bridging them. Removed a leftover 2.39 mm GND track that still touched
  J1.S2 and shorted straight across Q1.
- Add C12 470u/50V bulk and C13 0.1u HF bypass on +24V. C3 alone left the
  300 kHz - 100 MHz band uncovered while U4 switches at 500 kHz.
- Route the block: gate net kept inside 5 mm of Q1's gate; /GND1 return at
  1.50 mm (4.3 A capacity vs 1.85 A worst case through Q1).

Solenoid driver
- Add C25 0.1u across U1 pin 9 (COM) to GND. That node catches flyback from
  all seven channels and previously reached the +24V plane through ~50 mm of
  0.55 mm trace with nothing local.

Silkscreen
- Raise 403 graphic objects from 0.000/0.100/0.120/0.127 mm to the 0.15 mm
  fab minimum; five were zero-width, which is undefined behaviour. Fix one
  0.45 mm text height and one 0.09 mm stroke.
- Selector valve legend: label 'J23' named a part that does not exist; the
  connector there is J25. Recentre all 12 labels on their own connectors,
  strip stray newlines, and hide 7 duplicate footprint refdes that sat
  midway between connectors and read as shifted by one.

Cleanup
- Remove two /SDA and /SCL vias that connected B.Cu to B.Cu after those nets
  moved to the back layer, and split a +3.3V track so its end meets a
  junction rather than landing mid-span.
- Stitch an orphaned F.Cu ground island that had captured D3's cathode pad.

BOM
- Correct three MPNs that contradicted their own values and packages:
  R3 5.6k/0805 was a 680R 0603 part, R4 47k/0402 was a 4k7 0603 part,
  R5 3k/0402 was a 270R 0603 part.
- J1 car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
Parts:
- R39, R40: value 10k -> 2.2k
Changed lines of the file:
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@@
 			)
 		)
-		(property "Value" "10k"
+		(property "Value" "2.2k"
 			(at 156.21 81.28 0)
 			(show_name no)
@@
 		)
 		(instances
-			(project "fluidics-v2"
+			(project "fluidics-v3"
 				(path "/0ec91c42-8aad-437d-8c85-5e10f0e51fe0/b627bb7a-5c26-4d4a-8ee1-9b58f0107eeb"
 					(reference "R42")
@@
 			)
 		)
-		(property "Value" "10k"
+		(property "Value" "2.2k"
 			(at 140.97 78.74 0)
 			(show_name no)
@@
 		)
 		(instances
-			(project "fluidics-v2"
+			(project "fluidics-v3"
 				(path "/0ec91c42-8aad-437d-8c85-5e10f0e51fe0/b627bb7a-5c26-4d4a-8ee1-9b58f0107eeb"
 					(reference "R41")
@@
 		)
 		(instances
-			(project "fluidics-v2"
+			(project "fluidics-v3"
 				(path "/0ec91c42-8aad-437d-8c85-5e10f0e51fe0/b627bb7a-5c26-4d4a-8ee1-9b58f0107eeb"
 					(reference "#PWR0133")
@@
 		)
 		(instances
-			(project "fluidics-v2"
+			(project "fluidics-v3"
 				(path "/0ec91c42-8aad-437d-8c85-5e10f0e51fe0/b627bb7a-5c26-4d4a-8ee1-9b58f0107eeb"
 					(reference "#PWR0134")

Commit message: fab: apply JLCPCB part selections to BOM, annotate strays, normalise CPL
Sourcing
- Write Manufacturer_Part_Number / Manufacturer_Name / LCSC for every part
  from the JLCPCB BOM-matching sheet. 33 of 34 BOM rows now carry an LCSC
  code; the exception is J10/J12/J14/J18/J21/J25 (Molex 87832-0410), which
  JLCPCB returned "No matches" for and still needs a part chosen.

Substitutions accepted from the sheet
- IC2  ADuM1250WSRZ-RL7 -> ISO1640BDR (TI). Verified pin-for-pin against the
  board: 1 VCC1, 2 SDA1, 3 SCL1, 4 GND1, 5 GND2, 6 SCL2, 7 SDA2, 8 VCC2.
- C3   -> KEMET T521X336M050ATE050, which is 33uF/50V, not 100uF. Value
  updated to match. The 50 V rating fixes the derating problem the old
  unrated 100uF tantalum had on a 24 V rail; 33uF is ample now that C12
  carries 470uF ten millimetres away. Note the part is case X (7343-43,
  4.3 mm tall) against a footprint named 7343-20 - the land pattern is
  identical, only the height differs, and nothing sits above it.
- Q1   -> IRF540NPBF, J3 -> Connfly DS1037, D4 -> KT-0805R, J5 -> XY308.
- U13's MPN arrived truncated from JLCPCB as "TC7PZ17FU,LJ(CT"; restored the
  closing parenthesis.

Annotation
- D2/D3/D4, R3/R4/R5 (psu sheet) and H2/H3/H4 (root) were still unannotated
  "D?"/"R?"/"H?" symbols, so the BOM exporter was auto-numbering them on each
  run and no field edit could reach them. Annotated from the PCB footprint
  UUID paths rather than by position - H3 and H4 turned out to be the reverse
  of what their schematic coordinates suggested.

CPL
- Rotations now emitted 0-360; KiCad wrote 27 of them as negative (-90).
- Coordinates to 4 dp, rotation to 2 dp.
- BOM and CPL reconcile at 76 designators, no ranges, nothing one-sided.

ERC: 0 errors.

Co-Authored-By: Claude Opus 5 (1M context) <noreply@anthropic.com>
Parts:
- R39, R40: LCSC (none) -> C25879; Manufacturer_Name (none) -> UNI-ROYAL(Uniroyal Elec); Manufacturer_Part_Number (none) -> 0402WGF2201TCE
Changed lines of the file:
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@@
+			)
+		)
+		(property "LCSC" "C25879"
+			(at 0 0 0)
+			(hide yes)
+			(show_name no)
+			(do_not_autoplace no)
+			(effects
+				(font
+					(size 1.27 1.27)
+				)
+			)
+		)
+		(property "Manufacturer_Name" "UNI-ROYAL(Uniroyal Elec)"
+			(at 0 0 0)
+			(hide yes)
+			(show_name no)
+			(do_not_autoplace no)
+			(effects
+				(font
+					(size 1.27 1.27)
+				)
+			)
+		)
+		(property "Manufacturer_Part_Number" "0402WGF2201TCE"
+			(at 0 0 0)
+			(hide yes)
+			(show_name no)
+			(do_not_autoplace no)
+			(effects
+				(font
+					(size 1.27 1.27)
+				)
 			)
 		)
@@
 			)
 		)
+		(property "LCSC" "C25879"
+			(at 0 0 0)
+			(hide yes)
+			(show_name no)
+			(do_not_autoplace no)
+			(effects
+				(font
+					(size 1.27 1.27)
+				)
+			)
+		)
+		(property "Manufacturer_Name" "UNI-ROYAL(Uniroyal Elec)"
+			(at 0 0 0)
+			(hide yes)
+			(show_name no)
+			(do_not_autoplace no)
+			(effects
+				(font
+					(size 1.27 1.27)
+				)
+			)
+		)
+		(property "Manufacturer_Part_Number" "0402WGF2201TCE"
+			(at 0 0 0)
+			(hide yes)
+			(show_name no)
+			(do_not_autoplace no)
+			(effects
+				(font
+					(size 1.27 1.27)
+				)
+			)
+		)
