File: fluidics-v3/solenoid_driver.kicad_sch (KiCad schematic)
At the start: 3 parts, among them J5 Screw_Terminal_01x06, U1 TPL7407LDR

Commit message: fab: apply JLCPCB part selections to BOM, annotate strays, normalise CPL
Sourcing
- Write Manufacturer_Part_Number / Manufacturer_Name / LCSC for every part
  from the JLCPCB BOM-matching sheet. 33 of 34 BOM rows now carry an LCSC
  code; the exception is J10/J12/J14/J18/J21/J25 (Molex 87832-0410), which
  JLCPCB returned "No matches" for and still needs a part chosen.

Substitutions accepted from the sheet
- IC2  ADuM1250WSRZ-RL7 -> ISO1640BDR (TI). Verified pin-for-pin against the
  board: 1 VCC1, 2 SDA1, 3 SCL1, 4 GND1, 5 GND2, 6 SCL2, 7 SDA2, 8 VCC2.
- C3   -> KEMET T521X336M050ATE050, which is 33uF/50V, not 100uF. Value
  updated to match. The 50 V rating fixes the derating problem the old
  unrated 100uF tantalum had on a 24 V rail; 33uF is ample now that C12
  carries 470uF ten millimetres away. Note the part is case X (7343-43,
  4.3 mm tall) against a footprint named 7343-20 - the land pattern is
  identical, only the height differs, and nothing sits above it.
- Q1   -> IRF540NPBF, J3 -> Connfly DS1037, D4 -> KT-0805R, J5 -> XY308.
- U13's MPN arrived truncated from JLCPCB as "TC7PZ17FU,LJ(CT"; restored the
  closing parenthesis.

Annotation
- D2/D3/D4, R3/R4/R5 (psu sheet) and H2/H3/H4 (root) were still unannotated
  "D?"/"R?"/"H?" symbols, so the BOM exporter was auto-numbering them on each
  run and no field edit could reach them. Annotated from the PCB footprint
  UUID paths rather than by position - H3 and H4 turned out to be the reverse
  of what their schematic coordinates suggested.

CPL
- Rotations now emitted 0-360; KiCad wrote 27 of them as negative (-90).
- Coordinates to 4 dp, rotation to 2 dp.
- BOM and CPL reconcile at 76 designators, no ranges, nothing one-sided.

ERC: 0 errors.

Co-Authored-By: Claude Opus 5 (1M context) <noreply@anthropic.com>
Parts:
- C25: LCSC (none) -> C14663; Manufacturer_Name (none) -> YAGEO; Manufacturer_Part_Number (none) -> CC0603KRX7R9BB104
- J5: LCSC (none) -> C915915; Manufacturer_Name (none) -> Ningbo Xinlaiya Elec.; Manufacturer_Part_Number (none) -> XY308-2.54-6P
- U1: LCSC (none) -> C139663
Changed lines of the file:
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@@
+			)
+		)
+		(property "LCSC" "C139663"
+			(at 0 0 0)
+			(hide yes)
+			(show_name no)
+			(do_not_autoplace no)
+			(effects
+				(font
+					(size 1.27 1.27)
+				)
 			)
 		)
@@
 			)
 		)
+		(property "LCSC" "C14663"
+			(at 0 0 0)
+			(hide yes)
+			(show_name no)
+			(do_not_autoplace no)
+			(effects
+				(font
+					(size 1.27 1.27)
+				)
+			)
+		)
+		(property "Manufacturer_Name" "YAGEO"
+			(at 0 0 0)
+			(hide yes)
+			(show_name no)
+			(do_not_autoplace no)
+			(effects
+				(font
+					(size 1.27 1.27)
+				)
+			)
+		)
+		(property "Manufacturer_Part_Number" "CC0603KRX7R9BB104"
+			(at 0 0 0)
+			(hide yes)
+			(show_name no)
+			(do_not_autoplace no)
+			(effects
+				(font
+					(size 1.27 1.27)
+				)
+			)
+		)
 		(property "Footprint" "Capacitor_SMD:C_0603_1608Metric"
 			(at 139.7 120.65 0)
@@
 			)
 		)
+		(property "LCSC" "C915915"
+			(at 0 0 0)
+			(hide yes)
+			(show_name no)
+			(do_not_autoplace no)
+			(effects
+				(font
+					(size 1.27 1.27)
+				)
+			)
+		)
+		(property "Manufacturer_Name" "Ningbo Xinlaiya Elec."
+			(at 0 0 0)
+			(hide yes)
+			(show_name no)
+			(do_not_autoplace no)
+			(effects
+				(font
+					(size 1.27 1.27)
+				)
+			)
+		)
+		(property "Manufacturer_Part_Number" "XY308-2.54-6P"
+			(at 0 0 0)
+			(hide yes)
+			(show_name no)
+			(do_not_autoplace no)
+			(effects
+				(font
+					(size 1.27 1.27)
+				)
+			)
+		)
