File: fluidics-v3/svalves.kicad_sch (KiCad schematic)
At the start: 10 parts, among them IC2 ADUM1250WSRZ-RL7, U6 LTC4311CSC6-TRPBF

Commit message: v3 PCB: 3.3V power-plane islands + B.Cu bridge, refdes to F.Fab, block silk labels
PCB (this session, verified DRC-clean, 0 electrical regressions):
- Add +3.3V copper islands on In2.Cu (top U11/IC2 cluster + LDO/I2C-connector corner)
- Add +3.3V bridge pour on B.Cu down the inter-island corridor; delete ~18mm redundant vertical run
- Stitch 3.3V loads to islands with vias; remove ~35mm circuitous surface routing (3.3V trace 194->68mm)
- Move 21 hidden reference designators (caps, R22/R23/R51, U2 Teensy) to F.Fab, centered
- Add functional F.Silkscreen labels: Solenoid Driver, Flow, I2C Iso, RS-232

Also bundles accompanying schematic/library work not authored this session
(fluidics-v2.kicad_sch, svalves, solenoid_driver, 87832-0410 Molex connector lib).

Co-Authored-By: Claude Opus 4.8 (1M context) <noreply@anthropic.com>
Connections:
- net SCL 5V: no longer R1.1, U6.6 (BUS1)
- net SDA 5V: no longer R1.2, U6.4 (BUS2)
- new net: R1.1, U6.6 (BUS1)
- new net: R1.2, U6.4 (BUS2)
Changed lines of the file:
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@@
-	)
-	(junction
-		(at 110.49 78.74)
-		(diameter 0)
-		(color 0 0 0 0)
 	)
 	(junction
@@
 	)
 	(junction
-		(at 102.87 57.15)
-		(diameter 0)
-		(color 0 0 0 0)
-	)
-	(junction
-		(at 110.49 54.61)
-		(diameter 0)
-		(color 0 0 0 0)
-	)
-	(junction
 		(at 128.27 57.15)
 		(diameter 0)
@@
 	)
 	(junction
-		(at 102.87 78.74)
-		(diameter 0)
-		(color 0 0 0 0)
-	)
-	(junction
 		(at 124.46 54.61)
 		(diameter 0)
@@
 	(wire
 		(pts
-			(xy 102.87 78.74) (xy 102.87 57.15)
-		)
-		(stroke
-			(width 0)
-			(type default)
-		)
-	)
-	(wire
-		(pts
 			(xy 49.53 39.37) (xy 59.69 39.37)
 		)
@@
 	(wire
 		(pts
-			(xy 110.49 54.61) (xy 110.49 78.74)
-		)
-		(stroke
-			(width 0)
-			(type default)
-		)
-	)
-	(wire
-		(pts
 			(xy 107.95 46.99) (xy 97.79 46.99)
 		)
@@
 	(wire
 		(pts
-			(xy 102.87 57.15) (xy 128.27 57.15)
-		)
-		(stroke
-			(width 0)
-			(type default)
-		)
-	)
-	(wire
-		(pts
-			(xy 92.71 54.61) (xy 110.49 54.61)
+			(xy 92.71 54.61) (xy 124.46 54.61)
 		)
 		(stroke
@@
 	(wire
 		(pts
-			(xy 92.71 57.15) (xy 102.87 57.15)
+			(xy 92.71 57.15) (xy 128.27 57.15)
 		)
 		(stroke
@@
 		)
 		(stroke
-			(width 0)
-			(type default)
-		)
-	)
-	(wire
-		(pts
-			(xy 110.49 54.61) (xy 124.46 54.61)
-		)
-		(stroke

Commit message: DNP the orphaned LTC4311, clean the CPL, fix undersized silk text
U6 (LTC4311 I2C accelerator) and R1 (0R) are vestigial from the accelerator
removal and cannot work as placed: pcbnew connectivity shows U6.1/U6.3 are the
only two of the twenty +5V pads unreachable from the buck output U4.5, and the
bus pins connect solely to each other -- Net-(U6-BUS1) = {U6.6, R1.1},
Net-(U6-BUS2) = {U6.4, R1.2}. Marked DNP on both the schematic (svalves sheet)
and the board rather than deleted, so the copper is left untouched and the
choice is reversible; deleting both is the cleaner fix for a future revision.

H2/H3/H4 (mounting holes) and TP1/TP2/TP3 (test points) are not placeable
parts but were being emitted into the placement file. Marked exclude-from-
position-files. Position export now also passes --exclude-dnp, so the CPL
drops from 82 to 74 rows and contains only parts a machine actually places.

Silk text "+3.3V CAP" was 0.8 x 0.6 mm against the board's own 0.8 mm silk
minimum; height raised to 0.8 mm. DRC text_height 1 -> 0, no other violation
moved.

Verified after the change: 44/44 socket pins still on the correct net, 4/4
intended no-connects, DRC unconnected 6 (unchanged baseline), schematic parity
0, 0 electrical violations, cosmetic 85 -> 84. Fab package regenerated.

Co-Authored-By: Claude Opus 5 (1M context) <noreply@anthropic.com>
Parts:
- R1, U6: now not fitted
Changed lines of the file:
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@@
 		(on_board yes)
 		(in_pos_files yes)
-		(dnp no)
+		(dnp yes)
 		(property "Reference" "R1"
 			(at 106.426 73.66 90)
@@
 		(on_board yes)
 		(in_pos_files yes)
-		(dnp no)
+		(dnp yes)
 		(fields_autoplaced yes)
 		(property "Reference" "U6"

Commit message: v3: +24V soft-start front end, U1 COM bypass, silkscreen and BOM fixes
Power input stage
- Replace TH1 (10 ohm NTC) with a low-side N-channel soft-start: Q1 (F60N80,
  TO-220) with a 100k/68k gate divider (R2/R6) and 0.1u timing cap (C11).
  The NTC sat in series with the whole board and dissipated 1.5-10 W; at
  1.85 A it was already over a 7 mm disc's rating before any valve moved.
- Split ground: /GND1 (J1 shell + pin 2) is now separate from GND, with Q1
  bridging them. Removed a leftover 2.39 mm GND track that still touched
  J1.S2 and shorted straight across Q1.
- Add C12 470u/50V bulk and C13 0.1u HF bypass on +24V. C3 alone left the
  300 kHz - 100 MHz band uncovered while U4 switches at 500 kHz.
- Route the block: gate net kept inside 5 mm of Q1's gate; /GND1 return at
  1.50 mm (4.3 A capacity vs 1.85 A worst case through Q1).

Solenoid driver
- Add C25 0.1u across U1 pin 9 (COM) to GND. That node catches flyback from
  all seven channels and previously reached the +24V plane through ~50 mm of
  0.55 mm trace with nothing local.

Silkscreen
- Raise 403 graphic objects from 0.000/0.100/0.120/0.127 mm to the 0.15 mm
  fab minimum; five were zero-width, which is undefined behaviour. Fix one
  0.45 mm text height and one 0.09 mm stroke.
- Selector valve legend: label 'J23' named a part that does not exist; the
  connector there is J25. Recentre all 12 labels on their own connectors,
  strip stray newlines, and hide 7 duplicate footprint refdes that sat
  midway between connectors and read as shifted by one.

Cleanup
- Remove two /SDA and /SCL vias that connected B.Cu to B.Cu after those nets
  moved to the back layer, and split a +3.3V track so its end meets a
  junction rather than landing mid-span.
- Stitch an orphaned F.Cu ground island that had captured D3's cathode pad.

BOM
- Correct three MPNs that contradicted their own values and packages:
  R3 5.6k/0805 was a 680R 0603 part, R4 47k/0402 was a 4k7 0603 part,
  R5 3k/0402 was a 270R 0603 part.
- J1 car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
Parts:
- removed C6: 0.01u, Capacitor_SMD:C_0603_1608Metric, symbol Device:C
- removed R1: 0, Resistor_SMD:R_0402_1005Metric, symbol Device:R
- removed U6: LTC4311CSC6-TRPBF, LTC:SOT-6_SC_LIT-L, symbol LTC4311CSC6#TRPBF:LTC4311CSC6-TRPBF
- R22, R23: value 10k -> 2.2k
Other:
- note removed: "Active Pullup - increase number of devices connected at once and length of cable DNP this IC and check the signal integrity - only install if necessary"

Commit message: fab: apply JLCPCB part selections to BOM, annotate strays, normalise CPL
Sourcing
- Write Manufacturer_Part_Number / Manufacturer_Name / LCSC for every part
  from the JLCPCB BOM-matching sheet. 33 of 34 BOM rows now carry an LCSC
  code; the exception is J10/J12/J14/J18/J21/J25 (Molex 87832-0410), which
  JLCPCB returned "No matches" for and still needs a part chosen.

Substitutions accepted from the sheet
- IC2  ADuM1250WSRZ-RL7 -> ISO1640BDR (TI). Verified pin-for-pin against the
  board: 1 VCC1, 2 SDA1, 3 SCL1, 4 GND1, 5 GND2, 6 SCL2, 7 SDA2, 8 VCC2.
- C3   -> KEMET T521X336M050ATE050, which is 33uF/50V, not 100uF. Value
  updated to match. The 50 V rating fixes the derating problem the old
  unrated 100uF tantalum had on a 24 V rail; 33uF is ample now that C12
  carries 470uF ten millimetres away. Note the part is case X (7343-43,
  4.3 mm tall) against a footprint named 7343-20 - the land pattern is
  identical, only the height differs, and nothing sits above it.
- Q1   -> IRF540NPBF, J3 -> Connfly DS1037, D4 -> KT-0805R, J5 -> XY308.
- U13's MPN arrived truncated from JLCPCB as "TC7PZ17FU,LJ(CT"; restored the
  closing parenthesis.

Annotation
- D2/D3/D4, R3/R4/R5 (psu sheet) and H2/H3/H4 (root) were still unannotated
  "D?"/"R?"/"H?" symbols, so the BOM exporter was auto-numbering them on each
  run and no field edit could reach them. Annotated from the PCB footprint
  UUID paths rather than by position - H3 and H4 turned out to be the reverse
  of what their schematic coordinates suggested.

CPL
- Rotations now emitted 0-360; KiCad wrote 27 of them as negative (-90).
- Coordinates to 4 dp, rotation to 2 dp.
- BOM and CPL reconcile at 76 designators, no ranges, nothing one-sided.

ERC: 0 errors.

Co-Authored-By: Claude Opus 5 (1M context) <noreply@anthropic.com>
Parts:
- C5, C9: LCSC (none) -> C14663; Manufacturer_Name (none) -> YAGEO; Manufacturer_Part_Number (none) -> CC0603KRX7R9BB104
- C7, C8: LCSC (none) -> C28323; Manufacturer_Name (none) -> Samsung Electro-Mechanics; Manufacturer_Part_Number (none) -> CL21B105KBFNNNE
- IC2: LCSC (none) -> C5122339; Manufacturer_Name Analog Devices -> Texas Instruments; Manufacturer_Part_Number ADUM1250WSRZ-RL7 -> ISO1640BDR
- R22, R23: LCSC (none) -> C25879; Manufacturer_Name (none) -> UNI-ROYAL(Uniroyal Elec); Manufacturer_Part_Number (none) -> 0402WGF2201TCE
Changed lines of the file:
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@@
+			)
+		)
+		(property "LCSC" "C5122339"
+			(at 0 0 0)
+			(hide yes)
+			(show_name no)
+			(do_not_autoplace no)
+			(effects
+				(font
+					(size 1.27 1.27)
+				)
 			)
 		)
@@
 			)
 		)
-		(property "Manufacturer_Name" "Analog Devices"
+		(property "Manufacturer_Name" "Texas Instruments"
 			(at 88.9 59.69 0)
 			(hide yes)
@@
 			)
 		)
-		(property "Manufacturer_Part_Number" "ADUM1250WSRZ-RL7"
+		(property "Manufacturer_Part_Number" "ISO1640BDR"
 			(at 88.9 62.23 0)
 			(hide yes)
@@
 			)
 		)
+		(property "LCSC" "C14663"
+			(at 0 0 0)
+			(hide yes)
+			(show_name no)
+			(do_not_autoplace no)
+			(effects
+				(font
+					(size 1.27 1.27)
+				)
+			)
+		)
+		(property "Manufacturer_Name" "YAGEO"
+			(at 0 0 0)
+			(hide yes)
+			(show_name no)
+			(do_not_autoplace no)
+			(effects
+				(font
+					(size 1.27 1.27)
+				)
+			)
+		)
+		(property "Manufacturer_Part_Number" "CC0603KRX7R9BB104"
+			(at 0 0 0)
+			(hide yes)
+			(show_name no)
+			(do_not_autoplace no)
+			(effects
+				(font
+					(size 1.27 1.27)
+				)
+			)
+		)
 		(property "Footprint" "Capacitor_SMD:C_0603_1608Metric"
 			(at 50.4952 46.99 0)
@@
 				)
 				(justify left)
+			)
+		)
+		(property "LCSC" "C25879"
+			(at 0 0 0)
+			(hide yes)
+			(show_name no)
+			(do_not_autoplace no)
+			(effects
+				(font
+					(size 1.27 1.27)
+				)
+			)
+		)
+		(property "Manufacturer_Name" "UNI-ROYAL(Uniroyal Elec)"
+			(at 0 0 0)
+			(hide yes)
+			(show_name no)
+			(do_not_autoplace no)
+			(effects
+				(font
+					(size 1.27 1.27)
+				)
+			)
+		)
+		(property "Manufacturer_Part_Number" "0402WGF2201TCE"
+			(at 0 0 0)
+			(hide yes)
+			(show_name no)
+			(do_not_autoplace no)
+			(effects
+				(font
+					(size 1.27 1.27)
+				)
 			)
 		)
@@
 			)
 		)
+		(property "LCSC" "C28323"
+			(at 0 0 0)
+			(hide yes)
+			(show_name no)
+			(do_not_autoplace no)
+			(effects
+				(font
+					(size 1.27 1.27)
+				)
+			)
+		)
+		(property "Manufacturer_Name" "Samsung Electro-Mechanics"
+			(at 0 0 0)
+			(hide yes)
+			(show_name no)
+			(do_not_autoplace no)
+			(effects
+				(font
+					(size 1.27 1.27)
+				)
+			)
+		)
+		(property "Manufacturer_Part_Number" "CL21B105KBFNNNE"
+			(at 0 0 0)
+			(hide yes)
+			(show_name no)
+			(do_not_autoplace no)
+			(effects
+				(font
+					(size 1.27 1.27)
+				)
+			)
+		)
 		(property "Footprint" "Capacitor_SMD:C_0805_2012Metric"
 			(at 60.6552 46.99 0)
@@
 			)
 		)
+		(property "LCSC" "C28323"
+			(at 0 0 0)
+			(hide yes)
+			(show_name no)
+			(do_not_autoplace no)
+			(effects
+				(font
+					(size 1.27 1.27)
+				)
+			)
+		)
+		(property "Manufacturer_Name" "Samsung Electro-Mechanics"
+			(at 0 0 0)
+			(hide yes)
+			(show_name no)
+			(do_not_autoplace no)
+			(effects
+				(font
+					(size 1.27 1.27)
+				)
+			)
+		)
+		(property "Manufacturer_Part_Number" "CL21B105KBFNNNE"
+			(at 0 0 0)
+			(hide yes)
+			(show_name no)
+			(do_not_autoplace no)
+			(effects
+				(font
+					(size 1.27 1.27)
+				)
+			)
+		)
 		(property "Footprint" "Capacitor_SMD:C_0805_2012Metric"
 			(at 96.8248 46.99 0)
@@
 				)
 				(justify left)
+			)
+		)
+		(property "LCSC" "C25879"
+			(at 0 0 0)
+			(hide yes)
+			(show_name no)
+			(do_not_autoplace no)
+			(effects
+				(font
+					(size 1.27 1.27)
+				)
+			)
+		)
+		(property "Manufacturer_Name" "UNI-ROYAL(Uniroyal Elec)"
+			(at 0 0 0)
+			(hide yes)
+			(show_name no)
+			(do_not_autoplace no)
+			(effects
+				(font
+					(size 1.27 1.27)
+				)
+			)
+		)
+		(property "Manufacturer_Part_Number" "0402WGF2201TCE"
+			(at 0 0 0)
+			(hide yes)
+			(show_name no)
+			(do_not_autoplace no)
+			(effects
+				(font
+					(size 1.27 1.27)
+				)
 			)
 		)
@@
 			)
 		)
+		(property "LCSC" "C14663"
+			(at 0 0 0)
+			(hide yes)
+			(show_name no)
+			(do_not_autoplace no)
+			(effects
+				(font
+					(size 1.27 1.27)
+				)
+			)
+		)
+		(property "Manufacturer_Name" "YAGEO"
+			(at 0 0 0)
+			(hide yes)
+			(show_name no)
+			(do_not_autoplace no)
+			(effects
+				(font
+					(size 1.27 1.27)
+				)
+			)
+		)
+		(property "Manufacturer_Part_Number" "CC0603KRX7R9BB104"
+			(at 0 0 0)
+			(hide yes)
+			(show_name no)
+			(do_not_autoplace no)
+			(effects
+				(font
+					(size 1.27 1.27)
+				)
+			)
+		)
